Commit message: first steps

File: urdf/Carausius_Morosus.urdf (robot description, URDF)
Before this commit: robot Carausius_Morosus, 38 links, 37 joints
Links:
- removed link Abdomen_0
- removed link Abdomen_1
- removed link Abdomen_2
- removed link Abdomen_3
- removed link Carput
- removed link FL_CT_L
- removed link FL_CT_R
- removed link FL_Femur_L
- removed link FL_Femur_R
- removed link FL_Pretarsus_L
- removed link FL_Pretarsus_R
- removed link FL_Tarsus_L
- removed link FL_Tarsus_R
- removed link FL_Tibia_L
- removed link FL_Tibia_R
- removed link HL_CT_L
- removed link HL_CT_R
- removed link HL_Femur_L
- removed link HL_Femur_R
- removed link HL_Pretarsus_L
- removed link HL_Pretarsus_R
- removed link HL_Tarsus_L
- removed link HL_Tarsus_R
- removed link HL_Tibia_L
- removed link HL_Tibia_R
- removed link ML_CT_L
- removed link ML_CT_R
- removed link ML_Femur_L
- removed link ML_Femur_R
- removed link ML_Pretarsus_L
- removed link ML_Pretarsus_R
- removed link ML_Tarsus_L
- removed link ML_Tarsus_R
- removed link ML_Tibia_L
- removed link ML_Tibia_R
- removed link Mesothorax
- removed link Metathorax
- removed link Prothorax
- added link 01_Carput, mass 17.34; collision mesh filename=../meshes/dae/Textured_mesh_1.075.dae scale=1.0 1.0 1.0; visual mesh filename=../meshes/dae/Textured_mesh_1.dae scale=1.0 1.0 1.0
- added link 02_Prothorax, mass 16.52; collision mesh filename=../meshes/dae/Textured_mesh_1.038.dae scale=1.0 1.0 1.0; visual mesh filename=../meshes/dae/Textured_mesh_1.002.dae scale=1.0 1.0 1.0
- added link 03_Mesothorax, mass 106.97; collision mesh filename=../meshes/dae/Textured_mesh_1.064.dae scale=1.0 1.0 1.0; visual mesh filename=../meshes/dae/Textured_mesh_1.015.dae scale=1.0 1.0 1.0
- added link 04_Metathorax, mass 81.29; collision mesh filename=../meshes/dae/Textured_mesh_1.063.dae scale=1.0 1.0 1.0; visual mesh filename=../meshes/dae/Textured_mesh_1.025.dae scale=1.0 1.0 1.0
- added link 05_Abdomen_3, mass 80.68; collision mesh filename=../meshes/dae/Textured_mesh_1.062.dae scale=1.0 1.0 1.0; visual mesh filename=../meshes/dae/Textured_mesh_1.024.dae scale=1.0 1.0 1.0
- added link 06_Abdomen_2, mass 79.52; collision mesh filename=../meshes/dae/Textured_mesh_1.061.dae scale=1.0 1.0 1.0; visual mesh filename=../meshes/dae/Textured_mesh_1.035.dae scale=1.0 1.0 1.0
- added link 07_Abdomen_1, mass 54.07; collision mesh filename=../meshes/dae/Textured_mesh_1.060.dae scale=1.0 1.0 1.0; visual mesh filename=../meshes/dae/Textured_mesh_1.036.dae scale=1.0 1.0 1.0
- added link 08_Abdomen_0, mass 46.23; collision mesh filename=../meshes/dae/Textured_mesh_1.059.dae scale=1.0 1.0 1.0; visual mesh filename=../meshes/dae/Textured_mesh_1.037.dae scale=1.0 1.0 1.0
- added link 09_HL_CT_L, mass 1.05; collision mesh filename=../meshes/dae/Textured_mesh_1.053.dae scale=1.0 1.0 1.0; visual mesh filename=../meshes/dae/Textured_mesh_1.013.dae scale=1.0 1.0 1.0
- added link 10_HL_Femur_L, mass 4.5; collision mesh filename=../meshes/dae/Textured_mesh_1.049.dae scale=1.0 1.0 1.0; visual mesh filename=../meshes/dae/Textured_mesh_1.027.dae scale=1.0 1.0 1.0
- added link 11_HL_Tibia_L, mass 2.28; collision mesh filename=../meshes/dae/Textured_mesh_1.050.dae scale=1.0 1.0 1.0; visual mesh filename=../meshes/dae/Textured_mesh_1.029.dae scale=1.0 1.0 1.0
- added link 12_HL_Tarsus_L, mass 0.23; collision mesh filename=../meshes/dae/Textured_mesh_1.051.dae scale=1.0 1.0 1.0; visual mesh filename=../meshes/dae/Textured_mesh_1.028.dae scale=1.0 1.0 1.0
- added link 13_HL_Pretarsus_L, mass 0.3; collision mesh filename=../meshes/dae/Textured_mesh_1.052.dae scale=1.0 1.0 1.0; visual mesh filename=../meshes/dae/Textured_mesh_1.030.dae scale=1.0 1.0 1.0
- added link 14_HL_CT_R, mass 1.38; collision mesh filename=../meshes/dae/Textured_mesh_1.058.dae scale=1.0 1.0 1.0; visual mesh filename=../meshes/dae/Textured_mesh_1.026.dae scale=1.0 1.0 1.0
- added link 15_HL_Femur_R, mass 4.58; collision mesh filename=../meshes/dae/Textured_mesh_1.054.dae scale=1.0 1.0 1.0; visual mesh filename=../meshes/dae/Textured_mesh_1.031.dae scale=1.0 1.0 1.0
- added link 16_HL_Tibia_R, mass 1.99; collision mesh filename=../meshes/dae/Textured_mesh_1.055.dae scale=1.0 1.0 1.0; visual mesh filename=../meshes/dae/Textured_mesh_1.033.dae scale=1.0 1.0 1.0
- added link 17_HL_Tarsus_R, mass 0.33; collision mesh filename=../meshes/dae/Textured_mesh_1.056.dae scale=1.0 1.0 1.0; visual mesh filename=../meshes/dae/Textured_mesh_1.032.dae scale=1.0 1.0 1.0
- added link 18_HL_Pretarsus_R, mass 0.39; collision mesh filename=../meshes/dae/Textured_mesh_1.057.dae scale=1.0 1.0 1.0; visual mesh filename=../meshes/dae/Textured_mesh_1.034.dae scale=1.0 1.0 1.0
- added link 19_ML_CT_L, mass 0.88; collision mesh filename=../meshes/dae/Textured_mesh_1.048.dae scale=1.0 1.0 1.0; visual mesh filename=../meshes/dae/Textured_mesh_1.007.dae scale=1.0 1.0 1.0
- added link 20_ML_Femur_L, mass 4.57; collision mesh filename=../meshes/dae/Textured_mesh_1.044.dae scale=1.0 1.0 1.0; visual mesh filename=../meshes/dae/Textured_mesh_1.021.dae scale=1.0 1.0 1.0
- added link 21_ML_Tibia_L, mass 1.44; collision mesh filename=../meshes/dae/Textured_mesh_1.045.dae scale=1.0 1.0 1.0; visual mesh filename=../meshes/dae/Textured_mesh_1.022.dae scale=1.0 1.0 1.0
- added link 22_ML_Tarsus_L, mass 0.15; collision mesh filename=../meshes/dae/Textured_mesh_1.046.dae scale=1.0 1.0 1.0; visual mesh filename=../meshes/dae/Textured_mesh_1.023.dae scale=1.0 1.0 1.0
- added link 23_ML_Pretarsus_L, mass 0.18; collision mesh filename=../meshes/dae/Textured_mesh_1.047.dae scale=1.0 1.0 1.0; visual mesh filename=../meshes/dae/Textured_mesh_1.020.dae scale=1.0 1.0 1.0
- added link 24_ML_CT_R, mass 0.84; collision mesh filename=../meshes/dae/Textured_mesh_1.043.dae scale=1.0 1.0 1.0; visual mesh filename=../meshes/dae/Textured_mesh_1.014.dae scale=1.0 1.0 1.0
- added link 25_ML_Femur_R, mass 3.83; collision mesh filename=../meshes/dae/Textured_mesh_1.039.dae scale=1.0 1.0 1.0; visual mesh filename=../meshes/dae/Textured_mesh_1.016.dae scale=1.0 1.0 1.0
- added link 26_ML_Tibia_R, mass 1.49; collision mesh filename=../meshes/dae/Textured_mesh_1.040.dae scale=1.0 1.0 1.0; visual mesh filename=../meshes/dae/Textured_mesh_1.018.dae scale=1.0 1.0 1.0
- added link 27_ML_Tarsus_R, mass 0.23; collision mesh filename=../meshes/dae/Textured_mesh_1.041.dae scale=1.0 1.0 1.0; visual mesh filename=../meshes/dae/Textured_mesh_1.017.dae scale=1.0 1.0 1.0
- added link 28_ML_Pretarsus_R, mass 0.26; collision mesh filename=../meshes/dae/Textured_mesh_1.042.dae scale=1.0 1.0 1.0; visual mesh filename=../meshes/dae/Textured_mesh_1.019.dae scale=1.0 1.0 1.0
- added link 29_FL_CT_L, mass 1.28; collision mesh filename=../meshes/dae/Textured_mesh_1.069.dae scale=1.0 1.0 1.0; visual mesh filename=../meshes/dae/Textured_mesh_1.001.dae scale=1.0 1.0 1.0
- added link 30_FL_Femur_L, mass 6.69; collision mesh filename=../meshes/dae/Textured_mesh_1.068.dae scale=1.0 1.0 1.0; visual mesh filename=../meshes/dae/Textured_mesh_1.004.dae scale=1.0 1.0 1.0
- added link 31_FL_Tibia_L, mass 2.09; collision mesh filename=../meshes/dae/Textured_mesh_1.065.dae scale=1.0 1.0 1.0; visual mesh filename=../meshes/dae/Textured_mesh_1.005.dae scale=1.0 1.0 1.0
- added link 32_FL_Tarsus_L, mass 0.18; collision mesh filename=../meshes/dae/Textured_mesh_1.066.dae scale=1.0 1.0 1.0; visual mesh filename=../meshes/dae/Textured_mesh_1.003.dae scale=1.0 1.0 1.0
- added link 33_FL_Pretarsus_L, mass 0.27; collision mesh filename=../meshes/dae/Textured_mesh_1.067.dae scale=1.0 1.0 1.0; visual mesh filename=../meshes/dae/Textured_mesh_1.006.dae scale=1.0 1.0 1.0
- added link 34_FL_CT_R, mass 0.88; collision mesh filename=../meshes/dae/Textured_mesh_1.074.dae scale=1.0 1.0 1.0; visual mesh filename=../meshes/dae/Textured_mesh_1.008.dae scale=1.0 1.0 1.0
- added link 35_FL_Femur_R, mass 6.2; collision mesh filename=../meshes/dae/Textured_mesh_1.073.dae scale=1.0 1.0 1.0; visual mesh filename=../meshes/dae/Textured_mesh_1.010.dae scale=1.0 1.0 1.0
- added link 36_FL_Tibia_R, mass 2.64; collision mesh filename=../meshes/dae/Textured_mesh_1.070.dae scale=1.0 1.0 1.0; visual mesh filename=../meshes/dae/Textured_mesh_1.011.dae scale=1.0 1.0 1.0
- added link 37_FL_Tarsus_R, mass 0.17; collision mesh filename=../meshes/dae/Textured_mesh_1.071.dae scale=1.0 1.0 1.0; visual mesh filename=../meshes/dae/Textured_mesh_1.009.dae scale=1.0 1.0 1.0
- added link 38_FL_Pretarsus_R, mass 0.27; collision mesh filename=../meshes/dae/Textured_mesh_1.072.dae scale=1.0 1.0 1.0; visual mesh filename=../meshes/dae/Textured_mesh_1.012.dae scale=1.0 1.0 1.0
Joints:
- removed joint Abdomen_0
- removed joint Abdomen_1
- removed joint Abdomen_2
- removed joint Abdomen_3
- removed joint FL_CT_L
- removed joint FL_CT_R
- removed joint FL_Femur_L
- removed joint FL_Femur_R
- removed joint FL_Pretarsus_L
- removed joint FL_Pretarsus_R
- removed joint FL_Tarsus_L
- removed joint FL_Tarsus_R
- removed joint FL_Tibia_L
- removed joint FL_Tibia_R
- removed joint HL_CT_L
- removed joint HL_CT_R
- removed joint HL_Femur_L
- removed joint HL_Femur_R
- removed joint HL_Pretarsus_L
- removed joint HL_Pretarsus_R
- removed joint HL_Tarsus_L
- removed joint HL_Tarsus_R
- removed joint HL_Tibia_L
- removed joint HL_Tibia_R
- removed joint ML_CT_L
- removed joint ML_CT_R
- removed joint ML_Femur_L
- removed joint ML_Femur_R
- removed joint ML_Pretarsus_L
- removed joint ML_Pretarsus_R
- removed joint ML_Tarsus_L
- removed joint ML_Tarsus_R
- removed joint ML_Tibia_L
- removed joint ML_Tibia_R
- removed joint Mesothorax
- removed joint Metathorax
- removed joint Prothorax
- added joint 02_Prothorax: type revolute, parent 01_Carput, child 02_Prothorax, origin xyz=0 0 0 rpy=-1.5708 1.55593 -1.55593, axis 0 0 1.0, limit lower=-1.5708 upper=1.5708 effort=0 velocity=0
- added joint 03_Mesothorax: type revolute, parent 02_Prothorax, child 03_Mesothorax, origin xyz=-0.04181 0.35326 0.00516 rpy=0 0 0, axis 0 0 1.0, limit lower=-1.5708 upper=1.5708 effort=0 velocity=0
- added joint 04_Metathorax: type revolute, parent 03_Mesothorax, child 04_Metathorax, origin xyz=-0.0529 1.49806 0.0154 rpy=0 0 0, axis 0 0 1.0, limit lower=-1.5708 upper=1.5708 effort=0 velocity=0
- added joint 05_Abdomen_3: type revolute, parent 04_Metathorax, child 05_Abdomen_3, origin xyz=-0.04709 0.952 -0.01588 rpy=0 0 0, axis 0 0 1.0, limit lower=-1.5708 upper=1.5708 effort=0 velocity=0
- added joint 06_Abdomen_2: type revolute, parent 05_Abdomen_3, child 06_Abdomen_2, origin xyz=0.04239 0.84128 0.00484 rpy=0 0 0, axis 0 0 1.0, limit lower=-1.5708 upper=1.5708 effort=0 velocity=0
- added joint 07_Abdomen_1: type revolute, parent 06_Abdomen_2, child 07_Abdomen_1, origin xyz=0.00886 0.92056 0.01897 rpy=0 0 0, axis 0 0 1.0, limit lower=-1.5708 upper=1.5708 effort=0 velocity=0
- added joint 08_Abdomen_0: type revolute, parent 07_Abdomen_1, child 08_Abdomen_0, origin xyz=-0.01857 0.7985 -0.02414 rpy=0 0 0, axis 0 0 1.0, limit lower=-1.5708 upper=1.5708 effort=0 velocity=0
- added joint 09_HL_CT_L: type revolute, parent 04_Metathorax, child 09_HL_CT_L, origin xyz=0.11581 0.86767 0.17126 rpy=1.5708 -1.55593 -1.55593, axis 0 0 1.0, limit lower=-1.5708 upper=1.5708 effort=0 velocity=0
- added joint 10_HL_Femur_L: type revolute, parent 09_HL_CT_L, child 10_HL_Femur_L, origin xyz=0.11235 0.01234 0.00904 rpy=1.5708 0.01487 0.01487, axis 0 0 1.0, limit lower=-1.5708 upper=1.5708 effort=0 velocity=0
- added joint 11_HL_Tibia_L: type revolute, parent 10_HL_Femur_L, child 11_HL_Tibia_L, origin xyz=1.22244 0.01703 -0.00127 rpy=0 0 0, axis 0 0 1.0, limit lower=-1.5708 upper=1.5708 effort=0 velocity=0
- added joint 12_HL_Tarsus_L: type revolute, parent 11_HL_Tibia_L, child 12_HL_Tarsus_L, origin xyz=0.0317 -1.4681 -0.00568 rpy=0 0 0, axis 0 0 1.0, limit lower=-1.5708 upper=1.5708 effort=0 velocity=0
- added joint 13_HL_Pretarsus_L: type revolute, parent 12_HL_Tarsus_L, child 13_HL_Pretarsus_L, origin xyz=0.18012 -0.00329 -0.00104 rpy=0 0 0, axis 0 0 1.0, limit lower=-1.5708 upper=1.5708 effort=0 velocity=0
- added joint 14_HL_CT_R: type revolute, parent 04_Metathorax, child 14_HL_CT_R, origin xyz=0.05706 0.86858 -0.17293 rpy=1.5708 -1.55593 -1.55593, axis 0 0 1.0, limit lower=-1.5708 upper=1.5708 effort=0 velocity=0
- added joint 15_HL_Femur_R: type revolute, parent 14_HL_CT_R, child 15_HL_Femur_R, origin xyz=-0.13933 -0.00283 -0.00741 rpy=1.5708 0.01487 0.01487, axis 0 0 1.0, limit lower=-1.5708 upper=1.5708 effort=0 velocity=0
- added joint 16_HL_Tibia_R: type revolute, parent 15_HL_Femur_R, child 16_HL_Tibia_R, origin xyz=-1.2448 -0.07124 0.00429 rpy=0 0 0, axis 0 0 1.0, limit lower=-1.5708 upper=1.5708 effort=0 velocity=0
- added joint 17_HL_Tarsus_R: type revolute, parent 16_HL_Tibia_R, child 17_HL_Tarsus_R, origin xyz=0.00654 -1.27212 -0.00879 rpy=0 0 0, axis 0 0 1.0, limit lower=-1.5708 upper=1.5708 effort=0 velocity=0
- added joint 18_HL_Pretarsus_R: type revolute, parent 17_HL_Tarsus_R, child 18_HL_Pretarsus_R, origin xyz=-0.26774 -0.01534 0.01139 rpy=0 0 0, axis 0 0 1.0, limit lower=-1.5708 upper=1.5708 effort=0 velocity=0
- added joint 19_ML_CT_L: type revolute, parent 03_Mesothorax, child 19_ML_CT_L, origin xyz=0.05216 1.38959 0.19815 rpy=1.5708 -1.55593 -1.55593, axis 0 0 1.0, limit lower=-1.5708 upper=1.5708 effort=0 velocity=0
- added joint 20_ML_Femur_L: type revolute, parent 19_ML_CT_L, child 20_ML_Femur_L, origin xyz=0.12326 0.00677 -0.0102 rpy=1.5708 0.01487 0.01487, axis 0 0 1.0, limit lower=-1.5708 upper=1.5708 effort=0 velocity=0
- added joint 21_ML_Tibia_L: type revolute, parent 20_ML_Femur_L, child 21_ML_Tibia_L, origin xyz=1.02447 -0.02296 0.01027 rpy=0 0 0, axis 0 0 1.0, limit lower=-1.5708 upper=1.5708 effort=0 velocity=0
- added joint 22_ML_Tarsus_L: type revolute, parent 21_ML_Tibia_L, child 22_ML_Tarsus_L, origin xyz=0.0474 -1.12595 -0.00892 rpy=0 0 0, axis 0 0 1.0, limit lower=-1.5708 upper=1.5708 effort=0 velocity=0
- added joint 23_ML_Pretarsus_L: type revolute, parent 22_ML_Tarsus_L, child 23_ML_Pretarsus_L, origin xyz=0.16129 5e-05 -0.00209 rpy=0 0 0, axis 0 0 1.0, limit lower=-1.5708 upper=1.5708 effort=0 velocity=0
- added joint 24_ML_CT_R: type revolute, parent 03_Mesothorax, child 24_ML_CT_R, origin xyz=0.08834 1.4053 -0.14673 rpy=1.5708 -1.55593 -1.55593, axis 0 0 1.0, limit lower=-1.5708 upper=1.5708 effort=0 velocity=0
- added joint 25_ML_Femur_R: type revolute, parent 24_ML_CT_R, child 25_ML_Femur_R, origin xyz=-0.11998 0.00023 -0.00162 rpy=1.5708 0.01487 0.01487, axis 0 0 1.0, limit lower=-1.5708 upper=1.5708 effort=0 velocity=0
- added joint 26_ML_Tibia_R: type revolute, parent 25_ML_Femur_R, child 26_ML_Tibia_R, origin xyz=-1.00324 -0.01434 0.01466 rpy=0 0 0, axis 0 0 1.0, limit lower=-1.5708 upper=1.5708 effort=0 velocity=0
- added joint 27_ML_Tarsus_R: type revolute, parent 26_ML_Tibia_R, child 27_ML_Tarsus_R, origin xyz=-0.00804 -1.01475 0.00158 rpy=0 0 0, axis 0 0 1.0, limit lower=-1.5708 upper=1.5708 effort=0 velocity=0
- added joint 28_ML_Pretarsus_R: type revolute, parent 27_ML_Tarsus_R, child 28_ML_Pretarsus_R, origin xyz=-0.20934 -0.00253 -0.00584 rpy=0 0 0, axis 0 0 1.0, limit lower=-1.5708 upper=1.5708 effort=0 velocity=0
- added joint 29_FL_CT_L: type revolute, parent 02_Prothorax, child 29_FL_CT_L, origin xyz=0.01474 0.13803 0.12265 rpy=1.5708 -1.55593 -1.55593, axis 0 0 1.0, limit lower=-1.5708 upper=1.5708 effort=0 velocity=0
- added joint 30_FL_Femur_L: type revolute, parent 29_FL_CT_L, child 30_FL_Femur_L, origin xyz=0.12442 0.01758 -0.01703 rpy=1.5708 0.01487 0.01487, axis 0 0 1.0, limit lower=-1.5708 upper=1.5708 effort=0 velocity=0
- added joint 31_FL_Tibia_L: type revolute, parent 30_FL_Femur_L, child 31_FL_Tibia_L, origin xyz=1.39525 0.01628 -0.00914 rpy=0 0 0, axis 0 0 1.0, limit lower=-1.5708 upper=1.5708 effort=0 velocity=0
- added joint 32_FL_Tarsus_L: type revolute, parent 31_FL_Tibia_L, child 32_FL_Tarsus_L, origin xyz=0.02497 -1.29823 0.00154 rpy=0 0 0, axis 0 0 1.0, limit lower=-1.5708 upper=1.5708 effort=0 velocity=0
- added joint 33_FL_Pretarsus_L: type revolute, parent 32_FL_Tarsus_L, child 33_FL_Pretarsus_L, origin xyz=0.15796 -0.00992 -0.00606 rpy=0 0 0, axis 0 0 1.0, limit lower=-1.5708 upper=1.5708 effort=0 velocity=0
- added joint 34_FL_CT_R: type revolute, parent 02_Prothorax, child 34_FL_CT_R, origin xyz=0.02108 0.15758 -0.13854 rpy=1.5708 -1.55593 -1.55593, axis 0 0 1.0, limit lower=-1.5708 upper=1.5708 effort=0 velocity=0
- added joint 35_FL_Femur_R: type revolute, parent 34_FL_CT_R, child 35_FL_Femur_R, origin xyz=-0.10675 -0.00175 0.00476 rpy=1.5708 0.01487 0.01487, axis 0 0 1.0, limit lower=-1.5708 upper=1.5708 effort=0 velocity=0
- added joint 36_FL_Tibia_R: type revolute, parent 35_FL_Femur_R, child 36_FL_Tibia_R, origin xyz=-1.39541 -0.03843 0.00396 rpy=0 0 0, axis 0 0 1.0, limit lower=-1.5708 upper=1.5708 effort=0 velocity=0
- added joint 37_FL_Tarsus_R: type revolute, parent 36_FL_Tibia_R, child 37_FL_Tarsus_R, origin xyz=-0.00112 -1.41627 -0.00491 rpy=0 0 0, axis 0 0 1.0, limit lower=-1.5708 upper=1.5708 effort=0 velocity=0
- added joint 38_FL_Pretarsus_R: type revolute, parent 37_FL_Tarsus_R, child 38_FL_Pretarsus_R, origin xyz=-0.16119 -0.01761 -0.00282 rpy=0 0 0, axis 0 0 1.0, limit lower=-1.5708 upper=1.5708 effort=0 velocity=0
