Commit message: included texture

File: urdf/Carausius_Morosus.urdf (robot description, URDF)
Before this commit: robot Carausius_Morosus, 38 links, 37 joints
Links:
- link 01_Carput: geometry collision mesh filename=../meshes/obj/Textured_mesh_1.075.obj scale=1.0 1.0 1.0; visual mesh filename=../meshes/obj/Textured_mesh_1.obj scale=1.0 1.0 1.0
- link 02_Prothorax: geometry collision mesh filename=../meshes/obj/Textured_mesh_1.038.obj scale=1.0 1.0 1.0; visual mesh filename=../meshes/obj/Textured_mesh_1.002.obj scale=1.0 1.0 1.0
- link 03_Mesothorax: geometry collision mesh filename=../meshes/obj/Textured_mesh_1.064.obj scale=1.0 1.0 1.0; visual mesh filename=../meshes/obj/Textured_mesh_1.015.obj scale=1.0 1.0 1.0
- link 04_Metathorax: geometry collision mesh filename=../meshes/obj/Textured_mesh_1.063.obj scale=1.0 1.0 1.0; visual mesh filename=../meshes/obj/Textured_mesh_1.025.obj scale=1.0 1.0 1.0
- link 05_Abdomen_3: geometry collision mesh filename=../meshes/obj/Textured_mesh_1.062.obj scale=1.0 1.0 1.0; visual mesh filename=../meshes/obj/Textured_mesh_1.024.obj scale=1.0 1.0 1.0
- link 06_Abdomen_2: geometry collision mesh filename=../meshes/obj/Textured_mesh_1.061.obj scale=1.0 1.0 1.0; visual mesh filename=../meshes/obj/Textured_mesh_1.035.obj scale=1.0 1.0 1.0
- link 07_Abdomen_1: geometry collision mesh filename=../meshes/obj/Textured_mesh_1.060.obj scale=1.0 1.0 1.0; visual mesh filename=../meshes/obj/Textured_mesh_1.036.obj scale=1.0 1.0 1.0
- link 08_Abdomen_0: geometry collision mesh filename=../meshes/obj/Textured_mesh_1.059.obj scale=1.0 1.0 1.0; visual mesh filename=../meshes/obj/Textured_mesh_1.037.obj scale=1.0 1.0 1.0
- link 09_HL_CT_L: geometry collision mesh filename=../meshes/obj/Textured_mesh_1.053.obj scale=1.0 1.0 1.0; visual mesh filename=../meshes/obj/Textured_mesh_1.013.obj scale=1.0 1.0 1.0
- link 10_HL_Femur_L: geometry collision mesh filename=../meshes/obj/Textured_mesh_1.049.obj scale=1.0 1.0 1.0; visual mesh filename=../meshes/obj/Textured_mesh_1.027.obj scale=1.0 1.0 1.0
- link 11_HL_Tibia_L: geometry collision mesh filename=../meshes/obj/Textured_mesh_1.050.obj scale=1.0 1.0 1.0; visual mesh filename=../meshes/obj/Textured_mesh_1.029.obj scale=1.0 1.0 1.0
- link 12_HL_Tarsus_L: geometry collision mesh filename=../meshes/obj/Textured_mesh_1.051.obj scale=1.0 1.0 1.0; visual mesh filename=../meshes/obj/Textured_mesh_1.028.obj scale=1.0 1.0 1.0
- link 13_HL_Pretarsus_L: geometry collision mesh filename=../meshes/obj/Textured_mesh_1.052.obj scale=1.0 1.0 1.0; visual mesh filename=../meshes/obj/Textured_mesh_1.030.obj scale=1.0 1.0 1.0
- link 14_HL_CT_R: geometry collision mesh filename=../meshes/obj/Textured_mesh_1.058.obj scale=1.0 1.0 1.0; visual mesh filename=../meshes/obj/Textured_mesh_1.026.obj scale=1.0 1.0 1.0
- link 15_HL_Femur_R: geometry collision mesh filename=../meshes/obj/Textured_mesh_1.054.obj scale=1.0 1.0 1.0; visual mesh filename=../meshes/obj/Textured_mesh_1.031.obj scale=1.0 1.0 1.0
- link 16_HL_Tibia_R: geometry collision mesh filename=../meshes/obj/Textured_mesh_1.055.obj scale=1.0 1.0 1.0; visual mesh filename=../meshes/obj/Textured_mesh_1.033.obj scale=1.0 1.0 1.0
- link 17_HL_Tarsus_R: geometry collision mesh filename=../meshes/obj/Textured_mesh_1.056.obj scale=1.0 1.0 1.0; visual mesh filename=../meshes/obj/Textured_mesh_1.032.obj scale=1.0 1.0 1.0
- link 18_HL_Pretarsus_R: geometry collision mesh filename=../meshes/obj/Textured_mesh_1.057.obj scale=1.0 1.0 1.0; visual mesh filename=../meshes/obj/Textured_mesh_1.034.obj scale=1.0 1.0 1.0
- link 19_ML_CT_L: geometry collision mesh filename=../meshes/obj/Textured_mesh_1.048.obj scale=1.0 1.0 1.0; visual mesh filename=../meshes/obj/Textured_mesh_1.007.obj scale=1.0 1.0 1.0
- link 20_ML_Femur_L: geometry collision mesh filename=../meshes/obj/Textured_mesh_1.044.obj scale=1.0 1.0 1.0; visual mesh filename=../meshes/obj/Textured_mesh_1.021.obj scale=1.0 1.0 1.0
- link 21_ML_Tibia_L: geometry collision mesh filename=../meshes/obj/Textured_mesh_1.045.obj scale=1.0 1.0 1.0; visual mesh filename=../meshes/obj/Textured_mesh_1.022.obj scale=1.0 1.0 1.0
- link 22_ML_Tarsus_L: geometry collision mesh filename=../meshes/obj/Textured_mesh_1.046.obj scale=1.0 1.0 1.0; visual mesh filename=../meshes/obj/Textured_mesh_1.023.obj scale=1.0 1.0 1.0
- link 23_ML_Pretarsus_L: geometry collision mesh filename=../meshes/obj/Textured_mesh_1.047.obj scale=1.0 1.0 1.0; visual mesh filename=../meshes/obj/Textured_mesh_1.020.obj scale=1.0 1.0 1.0
- link 24_ML_CT_R: geometry collision mesh filename=../meshes/obj/Textured_mesh_1.043.obj scale=1.0 1.0 1.0; visual mesh filename=../meshes/obj/Textured_mesh_1.014.obj scale=1.0 1.0 1.0
- link 25_ML_Femur_R: geometry collision mesh filename=../meshes/obj/Textured_mesh_1.039.obj scale=1.0 1.0 1.0; visual mesh filename=../meshes/obj/Textured_mesh_1.016.obj scale=1.0 1.0 1.0
- link 26_ML_Tibia_R: geometry collision mesh filename=../meshes/obj/Textured_mesh_1.040.obj scale=1.0 1.0 1.0; visual mesh filename=../meshes/obj/Textured_mesh_1.018.obj scale=1.0 1.0 1.0
- link 27_ML_Tarsus_R: geometry collision mesh filename=../meshes/obj/Textured_mesh_1.041.obj scale=1.0 1.0 1.0; visual mesh filename=../meshes/obj/Textured_mesh_1.017.obj scale=1.0 1.0 1.0
- link 28_ML_Pretarsus_R: geometry collision mesh filename=../meshes/obj/Textured_mesh_1.042.obj scale=1.0 1.0 1.0; visual mesh filename=../meshes/obj/Textured_mesh_1.019.obj scale=1.0 1.0 1.0
- link 29_FL_CT_L: geometry collision mesh filename=../meshes/obj/Textured_mesh_1.069.obj scale=1.0 1.0 1.0; visual mesh filename=../meshes/obj/Textured_mesh_1.001.obj scale=1.0 1.0 1.0
- link 30_FL_Femur_L: geometry collision mesh filename=../meshes/obj/Textured_mesh_1.068.obj scale=1.0 1.0 1.0; visual mesh filename=../meshes/obj/Textured_mesh_1.004.obj scale=1.0 1.0 1.0
- link 31_FL_Tibia_L: geometry collision mesh filename=../meshes/obj/Textured_mesh_1.065.obj scale=1.0 1.0 1.0; visual mesh filename=../meshes/obj/Textured_mesh_1.005.obj scale=1.0 1.0 1.0
- link 32_FL_Tarsus_L: geometry collision mesh filename=../meshes/obj/Textured_mesh_1.066.obj scale=1.0 1.0 1.0; visual mesh filename=../meshes/obj/Textured_mesh_1.003.obj scale=1.0 1.0 1.0
- link 33_FL_Pretarsus_L: geometry collision mesh filename=../meshes/obj/Textured_mesh_1.067.obj scale=1.0 1.0 1.0; visual mesh filename=../meshes/obj/Textured_mesh_1.006.obj scale=1.0 1.0 1.0
- link 34_FL_CT_R: geometry collision mesh filename=../meshes/obj/Textured_mesh_1.074.obj scale=1.0 1.0 1.0; visual mesh filename=../meshes/obj/Textured_mesh_1.008.obj scale=1.0 1.0 1.0
- link 35_FL_Femur_R: geometry collision mesh filename=../meshes/obj/Textured_mesh_1.073.obj scale=1.0 1.0 1.0; visual mesh filename=../meshes/obj/Textured_mesh_1.010.obj scale=1.0 1.0 1.0
- link 36_FL_Tibia_R: geometry collision mesh filename=../meshes/obj/Textured_mesh_1.070.obj scale=1.0 1.0 1.0; visual mesh filename=../meshes/obj/Textured_mesh_1.011.obj scale=1.0 1.0 1.0
- link 37_FL_Tarsus_R: geometry collision mesh filename=../meshes/obj/Textured_mesh_1.071.obj scale=1.0 1.0 1.0; visual mesh filename=../meshes/obj/Textured_mesh_1.009.obj scale=1.0 1.0 1.0
- link 38_FL_Pretarsus_R: geometry collision mesh filename=../meshes/obj/Textured_mesh_1.072.obj scale=1.0 1.0 1.0; visual mesh filename=../meshes/obj/Textured_mesh_1.012.obj scale=1.0 1.0 1.0

Commit message: alles mögliche

File: urdf/Carausius_Morosus.urdf (robot description, URDF)
Before this commit: robot Carausius_Morosus, 38 links, 37 joints
Links:
- link 01_Carput: mass 17.34 -> 0.00173
- link 02_Prothorax: mass 16.52 -> 0.00165
- link 03_Mesothorax: mass 106.97 -> 0.0107
- link 04_Metathorax: mass 81.29 -> 0.00813
- link 05_Abdomen_3: mass 80.68 -> 0.00807
- link 06_Abdomen_2: mass 79.52 -> 0.00795
- link 07_Abdomen_1: mass 54.07 -> 0.00541
- link 08_Abdomen_0: mass 46.23 -> 0.00462
- link 09_HL_CT_L: mass 1.05 -> 0.0001
- link 10_HL_Femur_L: mass 4.5 -> 0.00045
- link 11_HL_Tibia_L: mass 2.28 -> 0.00023
- link 12_HL_Tarsus_L: mass 0.23 -> 2e-05
- link 13_HL_Pretarsus_L: mass 0.3 -> 3e-05
- link 14_HL_CT_R: mass 1.38 -> 0.00014
- link 15_HL_Femur_R: mass 4.58 -> 0.00046
- link 16_HL_Tibia_R: mass 1.99 -> 0.0002
- link 17_HL_Tarsus_R: mass 0.33 -> 3e-05
- link 18_HL_Pretarsus_R: mass 0.39 -> 4e-05
- link 19_ML_CT_L: mass 0.88 -> 9e-05
- link 20_ML_Femur_L: mass 4.57 -> 0.00046
- link 21_ML_Tibia_L: mass 1.44 -> 0.00014
- link 22_ML_Tarsus_L: mass 0.15 -> 1e-05
- link 23_ML_Pretarsus_L: mass 0.18 -> 2e-05
- link 24_ML_CT_R: mass 0.84 -> 8e-05
- link 25_ML_Femur_R: mass 3.83 -> 0.00038
- link 26_ML_Tibia_R: mass 1.49 -> 0.00015
- link 27_ML_Tarsus_R: mass 0.23 -> 2e-05
- link 28_ML_Pretarsus_R: mass 0.26 -> 3e-05
- link 29_FL_CT_L: mass 1.28 -> 0.00013
- link 30_FL_Femur_L: mass 6.69 -> 0.00067
- link 31_FL_Tibia_L: mass 2.09 -> 0.00021
- link 32_FL_Tarsus_L: mass 0.18 -> 2e-05
- link 33_FL_Pretarsus_L: mass 0.27 -> 3e-05
- link 34_FL_CT_R: mass 0.88 -> 9e-05
- link 35_FL_Femur_R: mass 6.2 -> 0.00062
- link 36_FL_Tibia_R: mass 2.64 -> 0.00026
- link 37_FL_Tarsus_R: mass 0.17 -> 2e-05
- link 38_FL_Pretarsus_R: mass 0.27 -> 3e-05
Joints:
- joint 09_HL_CT_L: origin xyz=0.11581 0.86767 0.17126 rpy=1.5708 -1.55593 -1.55593 -> xyz=0.11581 0.86767 0.17126 rpy=-1.5708 -1.06207 1.58566
- joint 14_HL_CT_R: origin xyz=0.05706 0.86858 -0.17293 rpy=1.5708 -1.55593 -1.55593 -> xyz=0.05706 0.86858 -0.17293 rpy=1.5708 -1.03233 -1.55593
- joint 29_FL_CT_L: origin xyz=0.01474 0.13803 0.12265 rpy=1.5708 -1.55593 -1.55593 -> xyz=0.01474 0.13803 0.12265 rpy=1.5708 -1.54344 -1.55593

Commit message: so einiges

File: urdf/Carausius_Morosus.urdf (robot description, URDF)
Before this commit: robot Carausius_Morosus, 38 links, 37 joints
Joints:
- joint 09_HL_CT_L: origin xyz=0.11581 0.86767 0.17126 rpy=-1.5708 -1.06207 1.58566 -> xyz=0.11581 0.86767 0.17126 rpy=-1.5708 -0.80027 1.58566
- joint 10_HL_Femur_L: origin xyz=0.11235 0.01234 0.00904 rpy=1.5708 0.01487 0.01487 -> xyz=0.11235 0.01234 0.00904 rpy=1.5708 -0.17679 0.01487
- joint 11_HL_Tibia_L: origin xyz=1.22244 0.01703 -0.00127 rpy=0 0 0 -> xyz=1.22244 0.01703 -0.00127 rpy=0 0 0.1853
- joint 12_HL_Tarsus_L: origin xyz=0.0317 -1.4681 -0.00568 rpy=0 0 0 -> xyz=0.0317 -1.4681 -0.00568 rpy=0 0 -0.35937
- joint 14_HL_CT_R: origin xyz=0.05706 0.86858 -0.17293 rpy=1.5708 -1.03233 -1.55593 -> xyz=0.05706 0.86858 -0.17293 rpy=1.5708 -0.77053 -1.55593
- joint 15_HL_Femur_R: origin xyz=-0.13933 -0.00283 -0.00741 rpy=1.5708 0.01487 0.01487 -> xyz=-0.13933 -0.00283 -0.00741 rpy=1.5708 0.34608 0.01487
- joint 16_HL_Tibia_R: origin xyz=-1.2448 -0.07124 0.00429 rpy=0 0 0 -> xyz=-1.2448 -0.07124 0.00429 rpy=0 0 0.09208
- joint 17_HL_Tarsus_R: origin xyz=0.00654 -1.27212 -0.00879 rpy=0 0 0 -> xyz=0.00654 -1.27212 -0.00879 rpy=0 0 0.15798
- joint 20_ML_Femur_L: origin xyz=0.12326 0.00677 -0.0102 rpy=1.5708 0.01487 0.01487 -> xyz=0.12326 0.00677 -0.0102 rpy=1.5708 -0.42082 0.01487
- joint 21_ML_Tibia_L: origin xyz=1.02447 -0.02296 0.01027 rpy=0 0 0 -> xyz=1.02447 -0.02296 0.01027 rpy=0 0 -0.28186
- joint 22_ML_Tarsus_L: origin xyz=0.0474 -1.12595 -0.00892 rpy=0 0 0 -> xyz=0.0474 -1.12595 -0.00892 rpy=0 0 -0.09032
- joint 25_ML_Femur_R: origin xyz=-0.11998 0.00023 -0.00162 rpy=1.5708 0.01487 0.01487 -> xyz=-0.11998 0.00023 -0.00162 rpy=1.5708 0.45666 0.01487
- joint 26_ML_Tibia_R: origin xyz=-1.00324 -0.01434 0.01466 rpy=0 0 0 -> xyz=-1.00324 -0.01434 0.01466 rpy=0 0 0.01545
- joint 27_ML_Tarsus_R: origin xyz=-0.00804 -1.01475 0.00158 rpy=0 0 0 -> xyz=-0.00804 -1.01475 0.00158 rpy=0 0 0.46229
- joint 29_FL_CT_L: origin xyz=0.01474 0.13803 0.12265 rpy=1.5708 -1.54344 -1.55593 -> xyz=0.01474 0.13803 0.12265 rpy=1.5708 -1.01984 -1.55593
- joint 30_FL_Femur_L: origin xyz=0.12442 0.01758 -0.01703 rpy=1.5708 0.01487 0.01487 -> xyz=0.12442 0.01758 -0.01703 rpy=1.57412 -0.24646 0.01448
- joint 31_FL_Tibia_L: origin xyz=1.39525 0.01628 -0.00914 rpy=0 0 0 -> xyz=1.39525 0.01628 -0.00914 rpy=0.00105 -0.00023 0.08576
- joint 34_FL_CT_R: origin xyz=0.02108 0.15758 -0.13854 rpy=1.5708 -1.55593 -1.55593 -> xyz=0.02108 0.15758 -0.13854 rpy=-1.5708 -1.06207 1.58566
- joint 35_FL_Femur_R: origin xyz=-0.10675 -0.00175 0.00476 rpy=1.5708 0.01487 0.01487 -> xyz=-0.10675 -0.00175 0.00476 rpy=1.5708 0.21853 0.01487
- joint 36_FL_Tibia_R: origin xyz=-1.39541 -0.03843 0.00396 rpy=0 0 0 -> xyz=-1.39541 -0.03843 0.00396 rpy=0 0 -0.18769
- joint 37_FL_Tarsus_R: origin xyz=-0.00112 -1.41627 -0.00491 rpy=0 0 0 -> xyz=-0.00112 -1.41627 -0.00491 rpy=0 0 0.37813
