Commit message: das ist alles

File: urdf/Carausius_Morosus.urdf (robot description, URDF)
Before this commit: robot Carausius_Morosus, 38 links, 37 joints
Links:
- removed link 05_Abdomen_3
- removed link 06_Abdomen_2
- removed link 07_Abdomen_1
- removed link 08_Abdomen_0
- removed link 09_HL_CT_L
- removed link 10_HL_Femur_L
- removed link 11_HL_Tibia_L
- removed link 12_HL_Tarsus_L
- removed link 13_HL_Pretarsus_L
- removed link 14_HL_CT_R
- removed link 15_HL_Femur_R
- removed link 16_HL_Tibia_R
- removed link 17_HL_Tarsus_R
- removed link 18_HL_Pretarsus_R
- removed link 19_ML_CT_L
- removed link 20_ML_Femur_L
- removed link 21_ML_Tibia_L
- removed link 22_ML_Tarsus_L
- removed link 23_ML_Pretarsus_L
- removed link 24_ML_CT_R
- removed link 25_ML_Femur_R
- removed link 26_ML_Tibia_R
- removed link 27_ML_Tarsus_R
- removed link 28_ML_Pretarsus_R
- removed link 29_FL_CT_L
- removed link 30_FL_Femur_L
- removed link 31_FL_Tibia_L
- removed link 32_FL_Tarsus_L
- removed link 33_FL_Pretarsus_L
- removed link 34_FL_CT_R
- removed link 35_FL_Femur_R
- removed link 36_FL_Tibia_R
- removed link 37_FL_Tarsus_R
- removed link 38_FL_Pretarsus_R
- added link 05_Abdomen3, mass 0.08065; collision box size=0.34948 0.84643 0.44251; visual mesh filename=../meshes/obj/Textured_mesh_1.024.obj scale=1.0 1.0 1.0
- added link 06_Abdomen2, mass 0.07952; collision box size=0.35343 0.92509 0.42333; visual mesh filename=../meshes/obj/Textured_mesh_1.035.obj scale=1.0 1.0 1.0
- added link 07_Abdomen1, mass 0.05407; collision box size=0.33276 0.80331 0.37792; visual mesh filename=../meshes/obj/Textured_mesh_1.036.obj scale=1.0 1.0 1.0
- added link 08_Abdomen0, mass 0.04623; collision box size=0.31676 0.7175 0.36188; visual mesh filename=../meshes/obj/Textured_mesh_1.037.obj scale=1.0 1.0 1.0
- added link 09_CT_HL_L, mass 0.00105; collision box size=0.11438 0.11821 0.15527; visual mesh filename=../meshes/obj/Textured_mesh_1.013.obj scale=1.0 1.0 1.0
- added link 10_Femur_HL_L, mass 0.0045; collision box size=1.2533 0.10548 0.12222; visual mesh filename=../meshes/obj/Textured_mesh_1.027.obj scale=1.0 1.0 1.0
- added link 11_Tibia_HL_L, mass 0.00283; collision box size=0.07513 0.0739 1.51698; visual mesh filename=../meshes/obj/Textured_mesh_1.029.obj scale=1.0 1.0 1.0
- added link 12_Tarsus_HL_L, mass 0.00053; collision box size=0.3786 0.09449 0.09233; visual mesh filename=../meshes/obj/Textured_mesh_1.030.obj scale=1.0 1.0 1.0
- added link 13_CT_HL_R, mass 0.00138; collision box size=0.1411 0.12043 0.16756; visual mesh filename=../meshes/obj/Textured_mesh_1.026.obj scale=1.0 1.0 1.0
- added link 14_Femur_HL_R, mass 0.00458; collision box size=1.27697 0.08758 0.1209; visual mesh filename=../meshes/obj/Textured_mesh_1.031.obj scale=1.0 1.0 1.0
- added link 15_Tibia_HL_R, mass 0.00199; collision box size=0.07538 0.07884 1.32637; visual mesh filename=../meshes/obj/Textured_mesh_1.033.obj scale=1.0 1.0 1.0
- added link 16_Tarsus_HL_R, mass 0.00072; collision box size=0.54248 0.09576 0.06815; visual mesh filename=../meshes/obj/Textured_mesh_1.032.obj scale=1.0 1.0 1.0
- added link 17_CT_ML_L, mass 0.00088; collision box size=0.12498 0.12881 0.13426; visual mesh filename=../meshes/obj/Textured_mesh_1.007.obj scale=1.0 1.0 1.0
- added link 18_Femur_ML_L, mass 0.00457; collision box size=1.04842 0.12186 0.10541; visual mesh filename=../meshes/obj/Textured_mesh_1.021.obj scale=1.0 1.0 1.0
- added link 19_Tibia_ML_L, mass 0.00144; collision box size=0.07714 0.07635 1.16387; visual mesh filename=../meshes/obj/Textured_mesh_1.022.obj scale=1.0 1.0 1.0
- added link 20_Tarsus_ML_L, mass 0.00034; collision box size=0.31035 0.09309 0.06525; visual mesh filename=../meshes/obj/Textured_mesh_1.020.obj scale=1.0 1.0 1.0
- added link 21_CT_ML_R, mass 0.00084; collision box size=0.12142 0.10543 0.14525; visual mesh filename=../meshes/obj/Textured_mesh_1.014.obj scale=1.0 1.0 1.0
- added link 22_Femur_ML_R, mass 0.00383; collision box size=1.03374 0.09225 0.13447; visual mesh filename=../meshes/obj/Textured_mesh_1.016.obj scale=1.0 1.0 1.0
- added link 23_Tibia_ML_R, mass 0.00149; collision box size=0.07381 0.06888 1.05127; visual mesh filename=../meshes/obj/Textured_mesh_1.018.obj scale=1.0 1.0 1.0
- added link 24_Tarsus_ML_R, mass 0.0005; collision box size=0.43172 0.09934 0.07049; visual mesh filename=../meshes/obj/Textured_mesh_1.017.obj scale=1.0 1.0 1.0
- added link 25_CT_FL_L, mass 0.00128; collision box size=0.12806 0.14832 0.16339; visual mesh filename=../meshes/obj/Textured_mesh_1.001.obj scale=1.0 1.0 1.0
- added link 26_Femur_FL_L, mass 0.00669; collision box size=1.4398 0.14697 0.13196; visual mesh filename=../meshes/obj/Textured_mesh_1.004.obj scale=1.0 1.0 1.0
- added link 27_Tibia_FL_L, mass 0.00209; collision box size=0.12238 0.08635 1.35634; visual mesh filename=../meshes/obj/Textured_mesh_1.005.obj scale=1.0 1.0 1.0
- added link 28_Tarsus_FL_L, mass 0.00045; collision box size=0.34782 0.06236 0.08457; visual mesh filename=../meshes/obj/Textured_mesh_1.006.obj scale=1.0 1.0 1.0
- added link 29_CT_FL_R, mass 0.00088; collision box size=0.10794 0.11094 0.14077; visual mesh filename=../meshes/obj/Textured_mesh_1.008.obj scale=1.0 1.0 1.0
- added link 30_Femur_FL_R, mass 0.0062; collision box size=1.42725 0.15388 0.12; visual mesh filename=../meshes/obj/Textured_mesh_1.010.obj scale=1.0 1.0 1.0
- added link 31_Tibia_FL_R, mass 0.00264; collision box size=0.10207 0.09593 1.45689; visual mesh filename=../meshes/obj/Textured_mesh_1.011.obj scale=1.0 1.0 1.0
- added link 32_Tarsus_FL_R, mass 0.00044; collision box size=0.35289 0.06335 0.08457; visual mesh filename=../meshes/obj/Textured_mesh_1.009.obj scale=1.0 1.0 1.0
- link 01_Carput: mass 17.34 -> 0.01734; geometry collision box size=0.2872 0.51114 0.26191; visual mesh filename=../meshes/obj/Textured_mesh_1.obj scale=1.0 1.0 1.0
- link 02_Prothorax: mass 16.52 -> 0.01652; geometry collision box size=0.26856 0.3839 0.2771; visual mesh filename=../meshes/obj/Textured_mesh_1.002.obj scale=1.0 1.0 1.0
- link 03_Mesothorax: mass 106.97 -> 0.107; geometry collision box size=0.35816 1.50299 0.41009; visual mesh filename=../meshes/obj/Textured_mesh_1.015.obj scale=1.0 1.0 1.0
- link 04_Metathorax: mass 81.29 -> 0.08129; geometry collision box size=0.35718 0.95917 0.40991; visual mesh filename=../meshes/obj/Textured_mesh_1.025.obj scale=1.0 1.0 1.0
Joints:
- removed joint 05_Abdomen_3
- removed joint 06_Abdomen_2
- removed joint 07_Abdomen_1
- removed joint 08_Abdomen_0
- removed joint 09_HL_CT_L
- removed joint 10_HL_Femur_L
- removed joint 11_HL_Tibia_L
- removed joint 12_HL_Tarsus_L
- removed joint 13_HL_Pretarsus_L
- removed joint 14_HL_CT_R
- removed joint 15_HL_Femur_R
- removed joint 16_HL_Tibia_R
- removed joint 17_HL_Tarsus_R
- removed joint 18_HL_Pretarsus_R
- removed joint 19_ML_CT_L
- removed joint 20_ML_Femur_L
- removed joint 21_ML_Tibia_L
- removed joint 22_ML_Tarsus_L
- removed joint 23_ML_Pretarsus_L
- removed joint 24_ML_CT_R
- removed joint 25_ML_Femur_R
- removed joint 26_ML_Tibia_R
- removed joint 27_ML_Tarsus_R
- removed joint 28_ML_Pretarsus_R
- removed joint 29_FL_CT_L
- removed joint 30_FL_Femur_L
- removed joint 31_FL_Tibia_L
- removed joint 32_FL_Tarsus_L
- removed joint 33_FL_Pretarsus_L
- removed joint 34_FL_CT_R
- removed joint 35_FL_Femur_R
- removed joint 36_FL_Tibia_R
- removed joint 37_FL_Tarsus_R
- removed joint 38_FL_Pretarsus_R
- added joint 05_Abdomen3: type revolute, parent 04_Metathorax, child 05_Abdomen3, origin xyz=-0.03293 0.95183 -0.01588 rpy=0 0 0, axis 0 0 1.0, limit lower=-1.0 upper=1.0 effort=0.05 velocity=5.0
- added joint 06_Abdomen2: type revolute, parent 05_Abdomen3, child 06_Abdomen2, origin xyz=0.05489 0.84056 0.00484 rpy=0 0 0, axis 0 0 1.0, limit lower=-1.0 upper=1.0 effort=0.05 velocity=5.0
- added joint 07_Abdomen1: type revolute, parent 06_Abdomen2, child 07_Abdomen1, origin xyz=0.02255 0.92033 0.01897 rpy=0 0 0, axis 0 0 1.0, limit lower=-1.0 upper=1.0 effort=0.05 velocity=5.0
- added joint 08_Abdomen0: type revolute, parent 07_Abdomen1, child 08_Abdomen0, origin xyz=-0.0067 0.79869 -0.02414 rpy=0 0 0, axis 0 0 1.0, limit lower=-1.0 upper=1.0 effort=0.05 velocity=5.0
- added joint 09_CT_HL_L: type revolute, parent 04_Metathorax, child 09_CT_HL_L, origin xyz=0.12869 0.86509 0.17126 rpy=-1.57079 -1.55219 1.57079, axis 0 0 1.0, limit lower=-1.0 upper=1.0 effort=0.05 velocity=5.0
- added joint 10_Femur_HL_L: type revolute, parent 09_CT_HL_L, child 10_Femur_HL_L, origin xyz=0.11252 0.01067 0.00904 rpy=-0.59697 -1.54968 2.15569, axis 0 0 1.0, limit lower=-1.0 upper=1.0 effort=0.05 velocity=5.0
- added joint 11_Tibia_HL_L: type revolute, parent 10_Femur_HL_L, child 11_Tibia_HL_L, origin xyz=1.22256 -0.00115 -0.00127 rpy=0.03004 0.00379 -1.4399, axis 0 0 1.0, limit lower=-1.0 upper=1.0 effort=0.05 velocity=5.0
- added joint 12_Tarsus_HL_L: type fixed, parent 11_Tibia_HL_L, child 12_Tarsus_HL_L, origin xyz=0.00987 -1.4684 -0.00568 rpy=-0.01177 0.00401 -0.15613
- added joint 13_CT_HL_R: type revolute, parent 04_Metathorax, child 13_CT_HL_R, origin xyz=0.06997 0.86687 -0.17293 rpy=1.5708 -0.7854 -1.5708, axis 0 0 1.0, limit lower=-1.0 upper=1.0 effort=0.05 velocity=5.0
- added joint 14_Femur_HL_R: type revolute, parent 13_CT_HL_R, child 14_Femur_HL_R, origin xyz=-0.13936 -0.00076 -0.00741 rpy=1.5708 0.49714 0, axis 0 0 1.0, limit lower=-1.0 upper=1.0 effort=0.05 velocity=5.0
- added joint 15_Tibia_HL_R: type revolute, parent 14_Femur_HL_R, child 15_Tibia_HL_R, origin xyz=-1.24572 -0.05273 0.00429 rpy=0 0 0, axis 0 0 1.0, limit lower=-1.0 upper=1.0 effort=0.05 velocity=5.0
- added joint 16_Tarsus_HL_R: type fixed, parent 15_Tibia_HL_R, child 16_Tarsus_HL_R, origin xyz=-0.01237 -1.27207 -0.00879 rpy=0 0 0.61847
- added joint 17_CT_ML_L: type revolute, parent 03_Mesothorax, child 17_CT_ML_L, origin xyz=0.07281 1.38866 0.19815 rpy=-1.5708 -1.0472 1.5708, axis 0 0 1.0, limit lower=-1.0 upper=1.0 effort=0.05 velocity=5.0
- added joint 18_Femur_ML_L: type revolute, parent 17_CT_ML_L, child 18_Femur_ML_L, origin xyz=0.12335 0.00493 -0.0102 rpy=1.5708 -0.46182 0, axis 0 0 1.0, limit lower=-1.0 upper=1.0 effort=500.0 velocity=100000000.0
- added joint 19_Tibia_ML_L: type revolute, parent 18_Femur_ML_L, child 19_Tibia_ML_L, origin xyz=1.02402 -0.03819 0.01027 rpy=0 0 -0.02841, axis 0 0 1.0, limit lower=-1.0 upper=1.0 effort=0.05 velocity=5.0
- added joint 20_Tarsus_ML_L: type fixed, parent 19_Tibia_ML_L, child 20_Tarsus_ML_L, origin xyz=0.03066 -1.12653 -0.00892 rpy=-0.00938 0.0069 -0.37586
- added joint 21_CT_ML_R: type revolute, parent 03_Mesothorax, child 21_CT_ML_R, origin xyz=0.10923 1.40383 -0.14673 rpy=-1.57078 -1.56507 1.57078, axis 0 0 1.0, limit lower=-1.0 upper=1.0 effort=0.05 velocity=5.0
- added joint 22_Femur_ML_R: type revolute, parent 21_CT_ML_R, child 22_Femur_ML_R, origin xyz=-0.11996 0.00201 -0.00162 rpy=1.22195 1.58592 -0.35207, axis 0 0 1.0, limit lower=-1.0 upper=1.0 effort=0.05 velocity=5.0
- added joint 23_Tibia_ML_R: type revolute, parent 22_Femur_ML_R, child 23_Tibia_ML_R, origin xyz=-1.00334 0.00058 0.01466 rpy=-0.0061 0.00169 1.31469, axis 0 0 1.0, limit lower=-1.0 upper=1.0 effort=0.05 velocity=5.0
- added joint 24_Tarsus_ML_R: type fixed, parent 23_Tibia_ML_R, child 24_Tarsus_ML_R, origin xyz=-0.02313 -1.01451 0.00158 rpy=0 0 0.26404
- added joint 25_CT_FL_L: type floating, parent 02_Prothorax, child 25_CT_FL_L, origin xyz=0.01679 0.13779 0.12265 rpy=0 -1.5708 0, limit effort=0.05 velocity=5.0
- added joint 26_Femur_FL_L: type revolute, parent 25_CT_FL_L, child 26_Femur_FL_L, origin xyz=0.12467 0.01607 -0.01596 rpy=1.5708 -1.56671 0, axis 0 0 1.0, limit lower=-1.0 upper=1.0 effort=0.05 velocity=5.0
- added joint 27_Tibia_FL_L: type revolute, parent 26_Femur_FL_L, child 27_Tibia_FL_L, origin xyz=1.39534 -0.00553 -0.00879 rpy=0 0 -1.41386, axis 0 0 1.0, limit lower=-1.0 upper=1.0 effort=0.05 velocity=5.0
- added joint 28_Tarsus_FL_L: type fixed, parent 27_Tibia_FL_L, child 28_Tarsus_FL_L, origin xyz=0.00566 -1.29846 0.00154 rpy=0 0 -0.47093
- added joint 29_CT_FL_R: type revolute, parent 02_Prothorax, child 29_CT_FL_R, origin xyz=0.02342 0.15725 -0.13854 rpy=-1.5708 -1.0472 1.5708, axis 0 0 1.0, limit lower=-1.0 upper=1.0 effort=0.05 velocity=5.0
- added joint 30_Femur_FL_R: type revolute, parent 29_CT_FL_R, child 30_Femur_FL_R, origin xyz=-0.10676 -0.00016 0.00476 rpy=1.5708 0.4962 0, axis 0 0 1.0, limit lower=-1.0 upper=1.0 effort=0.05 velocity=5.0
- added joint 31_Tibia_FL_R: type revolute, parent 30_Femur_FL_R, child 31_Tibia_FL_R, origin xyz=-1.39582 -0.01768 0.00396 rpy=0 0 0, axis 0 0 1.0, limit lower=-1.0 upper=1.0 effort=0.05 velocity=5.0
- added joint 32_Tarsus_FL_R: type fixed, parent 31_Tibia_FL_R, child 32_Tarsus_FL_R, origin xyz=-0.02218 -1.4161 -0.00491 rpy=0 0 0.57146
- joint 02_Prothorax: limit lower=-1.5708 upper=1.5708 effort=0 velocity=0 -> lower=-1.0 upper=1.0 effort=0.05 velocity=5.0; origin xyz=0 0 0 rpy=-1.5708 1.55593 -1.55593 -> xyz=0 0 0 rpy=0 0 0
- joint 03_Mesothorax: limit lower=-1.5708 upper=1.5708 effort=0 velocity=0 -> lower=-1.0 upper=1.0 effort=0.05 velocity=5.0; origin xyz=-0.04181 0.35326 0.00516 rpy=0 0 0 -> xyz=-0.03655 0.35385 0.00516 rpy=0 0 0
- joint 04_Metathorax: limit lower=-1.5708 upper=1.5708 effort=0 velocity=0 -> lower=-1.0 upper=1.0 effort=0.05 velocity=5.0; origin xyz=-0.0529 1.49806 0.0154 rpy=0 0 0 -> xyz=-0.03062 1.49945 0.0154 rpy=0 0 0
